Commit message: 1.12.0 Update the instructions and README.md about the local TM Robot corrected kinematics value loading and related codes.

File: tm_description/urdf/tm5-900.urdf (robot description, URDF)
Before this commit: robot tm5-900, 9 links, 8 joints
Links:
- link link_0: geometry collision mesh filename=package://tm_description/meshes/tm5-900/collision/tm5-base_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; visual mesh filename=package://tm_description/meshes/tm5-900/visual/tm5-base.obj
Joints:
- joint base_fixed_joint: origin xyz=0 0 0 rpy=0 0 0 -> xyz=0.000000 0.000000 0.000000 rpy=0.000000 0.000000 0.000000
- joint flange_fixed_joint: origin xyz=0 0 0 rpy=0 0 0 -> xyz=0.000000 0.000000 0.000000 rpy=0.000000 0.000000 0.000000
- joint joint_1: limit lower=-3.14 upper=3.14 effort=100.0 velocity=1.0 -> lower=-4.71238898038469 upper=4.71238898038469 effort=157 velocity=3.141592653589793; origin xyz=0 0 0.1452 rpy=0 0 0 -> xyz=0.000000 0.000000 0.145100 rpy=0.000000 -0.000000 0.000000
- joint joint_2: limit lower=-3.14 upper=3.14 effort=100.0 velocity=1.0 -> lower=-3.141592653589793 upper=3.141592653589793 effort=157 velocity=3.141592653589793; origin xyz=0 0 0 rpy=-1.570796327 -1.570796327 0 -> xyz=0.000000 0.000000 0.000000 rpy=-1.570796 -1.570796 0.000000
- joint joint_3: limit lower=-3.14 upper=3.14 effort=100.0 velocity=1.0 -> lower=-2.705260340591211 upper=2.705260340591211 effort=157 velocity=3.141592653589793; origin xyz=0.429 0 0 rpy=0 0 0 -> xyz=0.429000 0.000000 0.000000 rpy=0.000000 -0.000000 0.000000
- joint joint_4: limit lower=-3.14 upper=3.14 effort=10.0 velocity=1.0 -> lower=-3.141592653589793 upper=3.141592653589793 effort=43 velocity=3.9269908169872414; origin xyz=0.4115 0 -0.1223 rpy=0 0 1.570796327 -> xyz=0.411500 0.000000 -0.122200 rpy=0.000000 -0.000000 1.570796
- joint joint_5: limit lower=-3.14 upper=3.14 effort=10.0 velocity=1.0 -> lower=-3.141592653589793 upper=3.141592653589793 effort=43 velocity=3.9269908169872414; origin xyz=0 -0.106 0 rpy=1.570796327 0 0 -> xyz=0.000000 -0.106000 0.000000 rpy=1.570796 -0.000000 0.000000
- joint joint_6: limit lower=-3.14 upper=3.14 effort=10.0 velocity=1.0 -> lower=-4.71238898038469 upper=4.71238898038469 effort=43 velocity=3.9269908169872414; origin xyz=0 -0.11315 0 rpy=1.570796327 0 0 -> xyz=0.000000 -0.114400 0.000000 rpy=1.570796 -0.000000 0.000000

File: tm_description/xacro/macro.gazebo.xacro (robot description, xacro)
@@ -1,4 +1,4 @@
 <?xml version="1.0"?>
-<robot xmlns:xacro="http://wiki.ros.org/xacro">
+<robot xmlns:xacro="http://www.ros.org/wiki/xacro">
   <xacro:macro name="tmr_gazebo" params="ns prefix">
     <gazebo reference="${prefix}link_1">

File: tm_description/xacro/macro.inertial.xacro (robot description, xacro)
@@ -1,4 +1,4 @@
 <?xml version="1.0"?>
-<robot xmlns:xacro="http://wiki.ros.org/xacro">
+<robot xmlns:xacro="http://www.ros.org/wiki/xacro">
   <xacro:macro name="cylinder_inertial_x" params="radius length mass *origin">
     <inertial>
@@ -31,3 +31,13 @@
     </inertial>
   </xacro:macro>
+    <xacro:macro name="cuboid_inertial" params="width height depth mass *origin">
+    <inertial>
+      <mass value="${mass}" />
+      <xacro:insert_block name="origin" />
+      <inertia
+        ixx="${mass * (height * height + depth * depth) / 12}" ixy="0.0" ixz="0.0"
+        iyy="${mass * (width * width + height * height) / 12}" iyz="0.0"
+        izz="${mass * (width * width + depth * depth) / 12}" />
+    </inertial>
+  </xacro:macro>
 </robot>

File: tm_description/xacro/macro.materials.xacro (robot description, xacro)
@@ -2,6 +2,9 @@
 <robot xmlns:xacro="http://www.ros.org/wiki/xacro">
 	<xacro:macro name="tmr_materials">
-    <material name="grey">
+		<material name="lightgrey">
 			<color rgba="0.5 0.5 0.5 1.0" />
+		</material>
+		<material name="grey">
+			<color rgba="0.75 0.75 0.75 1.0" />
 		</material>
 		<material name="white">
@@ -32,4 +35,7 @@
 			<color rgba="0.0 0.0 0.0 1.0" />
 		</material>
+		<material name="darkolive">
+			<color rgba="0.3 0.3 0.25 1.0" />
+		</material>
 	</xacro:macro>
 </robot>

File: tm_description/xacro/macro.transmission.xacro (robot description, xacro)
@@ -1,4 +1,4 @@
 <?xml version="1.0"?>
-<robot xmlns:xacro="http://wiki.ros.org/xacro">
+<robot xmlns:xacro="http://www.ros.org/wiki/xacro">
   <xacro:macro name="tmr_transmission" params="prefix hw_iface">
     <transmission name="${prefix}trans_1">

File: tm_description/xacro/tm5-900.urdf.xacro (robot description, xacro)
@@ -1,7 +1,6 @@
 <?xml version="1.0"?>
-<robot xmlns:xacro="http://wiki.ros.org/xacro" name="tm5-900">
+<robot xmlns:xacro="http://www.ros.org/wiki/xacro" name="tm5-900">
   <xacro:arg name="ns" default="" />
   <xacro:arg name="prefix" default="" />
-  <xacro:arg name="gripper" default="none" />
   <xacro:arg name="color" default="none" />
   <xacro:arg name="trans_hw_iface" default="hardware_interface/PositionJointInterface" />
@@ -10,5 +9,7 @@
   <xacro:include filename="$(find tm_description)/xacro/macro.materials.xacro" />
   <!-- tm5-900 -->
-  <xacro:include filename="$(find tm_description)/xacro/macro.tm5-900.urdf.xacro" />
+  <!-- If the user want to use newly generated named robot description file as user_defined.urdf.xacro, -->
+  <!-- you must modify 'macro.tm5-900-nominal.urdf.xacro' to 'user_defined.urdf.xacro'  -->
+  <xacro:include filename="$(find tm_description)/xacro/macro.tm5-900-nominal.urdf.xacro" />
   <!--  -->
   <xacro:tmr_gazebo ns="$(arg ns)" prefix="$(arg prefix)" />
@@ -24,17 +25,3 @@
     <xacro:tm5-900 ns="$(arg ns)" prefix="$(arg prefix)" color="${color}" format="stl" />
   </xacro:unless>
-  <!-- Arm + Gripper -->
-  <xacro:property name="gripper" value="$(arg gripper)"/>
-  <xacro:if value="${gripper == 'robotiq_2f'}">
-    <xacro:include filename="$(find tm_description)/xacro/gripper/robotiq_2f.urdf.xacro" />
-    <xacro:robotiq_2f prefix="$(arg prefix)"/>
-  </xacro:if>
-<!--
-  <link name="world"/>
-  <joint name="world_joint" type="fixed">
-    <parent link="world" />
-    <child link="$(arg prefix)base"/>
-    <origin xyz="0 0 0" rpy="0 0 0"/>
-  </joint>
--->
 </robot>
