Commit message: 1.12.4 Update Link6 With camera, without camera interia parameters to Xacro, URDF files.

File: tm_description/urdf/tm12-nominal.urdf (robot description, URDF)
Before this commit: robot tm12, 9 links, 8 joints
Links:
- link link_6: mass 0.4 -> 0.65

File: tm_description/urdf/tm12x-nominal.urdf (robot description, URDF)
Before this commit: robot tm12x, 9 links, 8 joints
Links:
- link link_6: mass 0.4 -> 0.31

File: tm_description/urdf/tm14-nominal.urdf (robot description, URDF)
Before this commit: robot tm14, 9 links, 8 joints
Links:
- link link_6: mass 0.4 -> 0.65

File: tm_description/urdf/tm14x-nominal.urdf (robot description, URDF)
Before this commit: robot tm14x, 9 links, 8 joints
Links:
- link link_6: mass 0.4 -> 0.31

File: tm_description/urdf/tm5-700-nominal.urdf (robot description, URDF)
Before this commit: robot tm5-700, 9 links, 8 joints
Links:
- link link_6: mass 0.4 -> 0.65

File: tm_description/urdf/tm5-900-nominal.urdf (robot description, URDF)
Before this commit: robot tm5-900, 9 links, 8 joints
Links:
- link link_6: mass 0.4 -> 0.65

File: tm_description/urdf/tm5x-700-nominal.urdf (robot description, URDF)
Before this commit: robot tm5x-700, 9 links, 8 joints
Links:
- link link_6: mass 0.4 -> 0.31

File: tm_description/urdf/tm5x-900-nominal.urdf (robot description, URDF)
Before this commit: robot tm5x-900, 9 links, 8 joints
Links:
- link link_6: mass 0.4 -> 0.31

File: tm_description/xacro/macro.tm12-nominal.urdf.xacro (robot description, xacro)
@@ -44,5 +44,5 @@
     <xacro:property name="mass_4" value="1.576" />
     <xacro:property name="mass_5" value="1.576" />
-    <xacro:property name="mass_6" value="0.4" />
+    <xacro:property name="mass_6" value="0.65" />
     <xacro:property name="unit_factor" value="0.000001"/>
     <xacro:property name="ixx_1" value="${20289.334*unit_factor}" />
@@ -51,5 +51,5 @@
     <xacro:property name="ixx_4" value="${2058.405*unit_factor}" />
     <xacro:property name="ixx_5" value="${2058.405*unit_factor}" />
-    <xacro:property name="ixx_6" value="${476.643*unit_factor}" />
+    <xacro:property name="ixx_6" value="${774.544*unit_factor}" />
     <xacro:property name="iyy_1" value="${20289.334*unit_factor}" />
     <xacro:property name="iyy_2" value="${1175878.900*unit_factor}" />
@@ -57,5 +57,5 @@
     <xacro:property name="iyy_4" value="${2563.079*unit_factor}" />
     <xacro:property name="iyy_5" value="${2563.079*unit_factor}" />
-    <xacro:property name="iyy_6" value="${851.576*unit_factor}" />
+    <xacro:property name="iyy_6" value="${1383.811*unit_factor}" />
     <xacro:property name="izz_1" value="${21396.271*unit_factor}" />
     <xacro:property name="izz_2" value="${1203393.300*unit_factor}" />
@@ -63,5 +63,5 @@
     <xacro:property name="izz_4" value="${2643.21*unit_factor}" />
     <xacro:property name="izz_5" value="${2643.21*unit_factor}" />
-    <xacro:property name="izz_6" value="${959.69*unit_factor}" />
+    <xacro:property name="izz_6" value="${1559.496*unit_factor}" />
 <!--LinkDescription-->
   <link name="${prefix}link_0">

File: tm_description/xacro/macro.tm12x-nominal.urdf.xacro (robot description, xacro)
@@ -44,5 +44,5 @@
     <xacro:property name="mass_4" value="1.576" />
     <xacro:property name="mass_5" value="1.576" />
-    <xacro:property name="mass_6" value="0.4" />
+    <xacro:property name="mass_6" value="0.31" />
     <xacro:property name="unit_factor" value="0.000001"/>
     <xacro:property name="ixx_1" value="${20289.334*unit_factor}" />
@@ -51,5 +51,5 @@
     <xacro:property name="ixx_4" value="${2058.405*unit_factor}" />
     <xacro:property name="ixx_5" value="${2058.405*unit_factor}" />
-    <xacro:property name="ixx_6" value="${476.643*unit_factor}" />
+    <xacro:property name="ixx_6" value="${226.642*unit_factor}" />
     <xacro:property name="iyy_1" value="${20289.334*unit_factor}" />
     <xacro:property name="iyy_2" value="${1175878.900*unit_factor}" />
@@ -57,5 +57,5 @@
     <xacro:property name="iyy_4" value="${2563.079*unit_factor}" />
     <xacro:property name="iyy_5" value="${2563.079*unit_factor}" />
-    <xacro:property name="iyy_6" value="${851.576*unit_factor}" />
+    <xacro:property name="iyy_6" value="${226.642*unit_factor}" />
     <xacro:property name="izz_1" value="${21396.271*unit_factor}" />
     <xacro:property name="izz_2" value="${1203393.300*unit_factor}" />
@@ -63,5 +63,5 @@
     <xacro:property name="izz_4" value="${2643.21*unit_factor}" />
     <xacro:property name="izz_5" value="${2643.21*unit_factor}" />
-    <xacro:property name="izz_6" value="${959.69*unit_factor}" />
+    <xacro:property name="izz_6" value="${286.595*unit_factor}" />
 <!--LinkDescription-->
   <link name="${prefix}link_0">

File: tm_description/xacro/macro.tm14-nominal.urdf.xacro (robot description, xacro)
@@ -44,5 +44,5 @@
     <xacro:property name="mass_4" value="1.576" />
     <xacro:property name="mass_5" value="1.576" />
-    <xacro:property name="mass_6" value="0.4" />
+    <xacro:property name="mass_6" value="0.65" />
     <xacro:property name="unit_factor" value="0.000001"/>
     <xacro:property name="ixx_1" value="${20289.334*unit_factor}" />
@@ -51,5 +51,5 @@
     <xacro:property name="ixx_4" value="${2058.405*unit_factor}" />
     <xacro:property name="ixx_5" value="${2058.405*unit_factor}" />
-    <xacro:property name="ixx_6" value="${476.643*unit_factor}" />
+    <xacro:property name="ixx_6" value="${774.544*unit_factor}" />
     <xacro:property name="iyy_1" value="${20289.334*unit_factor}" />
     <xacro:property name="iyy_2" value="${1175878.900*unit_factor}" />
@@ -57,5 +57,5 @@
     <xacro:property name="iyy_4" value="${2563.079*unit_factor}" />
     <xacro:property name="iyy_5" value="${2563.079*unit_factor}" />
-    <xacro:property name="iyy_6" value="${851.576*unit_factor}" />
+    <xacro:property name="iyy_6" value="${1383.811*unit_factor}" />
     <xacro:property name="izz_1" value="${21396.271*unit_factor}" />
     <xacro:property name="izz_2" value="${1203393.300*unit_factor}" />
@@ -63,5 +63,5 @@
     <xacro:property name="izz_4" value="${2643.21*unit_factor}" />
     <xacro:property name="izz_5" value="${2643.21*unit_factor}" />
-    <xacro:property name="izz_6" value="${959.69*unit_factor}" />
+    <xacro:property name="izz_6" value="${1559.496*unit_factor}" />
 <!--LinkDescription-->
   <link name="${prefix}link_0">

File: tm_description/xacro/macro.tm14x-nominal.urdf.xacro (robot description, xacro)
@@ -44,5 +44,5 @@
     <xacro:property name="mass_4" value="1.576" />
     <xacro:property name="mass_5" value="1.576" />
-    <xacro:property name="mass_6" value="0.4" />
+    <xacro:property name="mass_6" value="0.31" />
     <xacro:property name="unit_factor" value="0.000001"/>
     <xacro:property name="ixx_1" value="${20289.334*unit_factor}" />
@@ -51,5 +51,5 @@
     <xacro:property name="ixx_4" value="${2058.405*unit_factor}" />
     <xacro:property name="ixx_5" value="${2058.405*unit_factor}" />
-    <xacro:property name="ixx_6" value="${476.643*unit_factor}" />
+    <xacro:property name="ixx_6" value="${226.642*unit_factor}" />
     <xacro:property name="iyy_1" value="${20289.334*unit_factor}" />
     <xacro:property name="iyy_2" value="${1175878.900*unit_factor}" />
@@ -57,5 +57,5 @@
     <xacro:property name="iyy_4" value="${2563.079*unit_factor}" />
     <xacro:property name="iyy_5" value="${2563.079*unit_factor}" />
-    <xacro:property name="iyy_6" value="${851.576*unit_factor}" />
+    <xacro:property name="iyy_6" value="${226.642*unit_factor}" />
     <xacro:property name="izz_1" value="${21396.271*unit_factor}" />
     <xacro:property name="izz_2" value="${1203393.300*unit_factor}" />
@@ -63,5 +63,5 @@
     <xacro:property name="izz_4" value="${2643.21*unit_factor}" />
     <xacro:property name="izz_5" value="${2643.21*unit_factor}" />
-    <xacro:property name="izz_6" value="${959.69*unit_factor}" />
+    <xacro:property name="izz_6" value="${286.595*unit_factor}" />
 <!--LinkDescription-->
   <link name="${prefix}link_0">

File: tm_description/xacro/macro.tm5-700-nominal.urdf.xacro (robot description, xacro)
@@ -44,5 +44,5 @@
     <xacro:property name="mass_4" value="1.576" />
     <xacro:property name="mass_5" value="1.576" />
-    <xacro:property name="mass_6" value="0.4" />
+    <xacro:property name="mass_6" value="0.65" />
     <xacro:property name="unit_factor" value="0.000001"/>
     <xacro:property name="ixx_1" value="${8800.119*unit_factor}" />
@@ -51,5 +51,5 @@
     <xacro:property name="ixx_4" value="${2058.405*unit_factor}" />
     <xacro:property name="ixx_5" value="${2058.405*unit_factor}" />
-    <xacro:property name="ixx_6" value="${476.643*unit_factor}" />
+    <xacro:property name="ixx_6" value="${774.544*unit_factor}" />
     <xacro:property name="iyy_1" value="${11548.982*unit_factor}" />
     <xacro:property name="iyy_2" value="${198251.97*unit_factor}" />
@@ -57,5 +57,5 @@
     <xacro:property name="iyy_4" value="${2563.079*unit_factor}" />
     <xacro:property name="iyy_5" value="${2563.079*unit_factor}" />
-    <xacro:property name="iyy_6" value="${851.576*unit_factor}" />
+    <xacro:property name="iyy_6" value="${1383.811*unit_factor}" />
     <xacro:property name="izz_1" value="${11970.081*unit_factor}" />
     <xacro:property name="izz_2" value="${204592.54*unit_factor}" />
@@ -63,5 +63,5 @@
     <xacro:property name="izz_4" value="${2643.21*unit_factor}" />
     <xacro:property name="izz_5" value="${2643.21*unit_factor}" />
-    <xacro:property name="izz_6" value="${959.69*unit_factor}" />
+    <xacro:property name="izz_6" value="${1559.496*unit_factor}" />
 <!--LinkDescription-->
   <link name="${prefix}link_0">

File: tm_description/xacro/macro.tm5-900-nominal.urdf.xacro (robot description, xacro)
@@ -44,5 +44,5 @@
     <xacro:property name="mass_4" value="1.576" />
     <xacro:property name="mass_5" value="1.576" />
-    <xacro:property name="mass_6" value="0.4" />
+    <xacro:property name="mass_6" value="0.65" />
     <xacro:property name="unit_factor" value="0.000001"/>
     <xacro:property name="ixx_1" value="${8800.119*unit_factor}" />
@@ -51,5 +51,5 @@
     <xacro:property name="ixx_4" value="${2058.405*unit_factor}" />
     <xacro:property name="ixx_5" value="${2058.405*unit_factor}" />
-    <xacro:property name="ixx_6" value="${476.643*unit_factor}" />
+    <xacro:property name="ixx_6" value="${774.544*unit_factor}" />
     <xacro:property name="iyy_1" value="${11548.982*unit_factor}" />
     <xacro:property name="iyy_2" value="${205888.616*unit_factor}" />
@@ -57,5 +57,5 @@
     <xacro:property name="iyy_4" value="${2563.079*unit_factor}" />
     <xacro:property name="iyy_5" value="${2563.079*unit_factor}" />
-    <xacro:property name="iyy_6" value="${851.576*unit_factor}" />
+    <xacro:property name="iyy_6" value="${1383.811*unit_factor}" />
     <xacro:property name="izz_1" value="${11970.081*unit_factor}" />
     <xacro:property name="izz_2" value="${212473.4246*unit_factor}" />
@@ -63,5 +63,5 @@
     <xacro:property name="izz_4" value="${2643.21*unit_factor}" />
     <xacro:property name="izz_5" value="${2643.21*unit_factor}" />
-    <xacro:property name="izz_6" value="${959.69*unit_factor}" />
+    <xacro:property name="izz_6" value="${1559.496*unit_factor}" />
 <!--LinkDescription-->
   <link name="${prefix}link_0">

File: tm_description/xacro/macro.tm5x-700-nominal.urdf.xacro (robot description, xacro)
@@ -44,5 +44,5 @@
     <xacro:property name="mass_4" value="1.576" />
     <xacro:property name="mass_5" value="1.576" />
-    <xacro:property name="mass_6" value="0.4" />
+    <xacro:property name="mass_6" value="0.31" />
     <xacro:property name="unit_factor" value="0.000001"/>
     <xacro:property name="ixx_1" value="${8800.119*unit_factor}" />
@@ -51,5 +51,5 @@
     <xacro:property name="ixx_4" value="${2058.405*unit_factor}" />
     <xacro:property name="ixx_5" value="${2058.405*unit_factor}" />
-    <xacro:property name="ixx_6" value="${476.643*unit_factor}" />
+    <xacro:property name="ixx_6" value="${226.642*unit_factor}" />
     <xacro:property name="iyy_1" value="${11548.982*unit_factor}" />
     <xacro:property name="iyy_2" value="${198251.97*unit_factor}" />
@@ -57,5 +57,5 @@
     <xacro:property name="iyy_4" value="${2563.079*unit_factor}" />
     <xacro:property name="iyy_5" value="${2563.079*unit_factor}" />
-    <xacro:property name="iyy_6" value="${851.576*unit_factor}" />
+    <xacro:property name="iyy_6" value="${226.642*unit_factor}" />
     <xacro:property name="izz_1" value="${11970.081*unit_factor}" />
     <xacro:property name="izz_2" value="${204592.54*unit_factor}" />
@@ -63,5 +63,5 @@
     <xacro:property name="izz_4" value="${2643.21*unit_factor}" />
     <xacro:property name="izz_5" value="${2643.21*unit_factor}" />
-    <xacro:property name="izz_6" value="${959.69*unit_factor}" />
+    <xacro:property name="izz_6" value="${286.595*unit_factor}" />
 <!--LinkDescription-->
   <link name="${prefix}link_0">

File: tm_description/xacro/macro.tm5x-900-nominal.urdf.xacro (robot description, xacro)
@@ -44,5 +44,5 @@
     <xacro:property name="mass_4" value="1.576" />
     <xacro:property name="mass_5" value="1.576" />
-    <xacro:property name="mass_6" value="0.4" />
+    <xacro:property name="mass_6" value="0.31" />
     <xacro:property name="unit_factor" value="0.000001"/>
     <xacro:property name="ixx_1" value="${8800.119*unit_factor}" />
@@ -51,5 +51,5 @@
     <xacro:property name="ixx_4" value="${2058.405*unit_factor}" />
     <xacro:property name="ixx_5" value="${2058.405*unit_factor}" />
-    <xacro:property name="ixx_6" value="${476.643*unit_factor}" />
+    <xacro:property name="ixx_6" value="${226.642*unit_factor}" />
     <xacro:property name="iyy_1" value="${11548.982*unit_factor}" />
     <xacro:property name="iyy_2" value="${205888.616*unit_factor}" />
@@ -57,5 +57,5 @@
     <xacro:property name="iyy_4" value="${2563.079*unit_factor}" />
     <xacro:property name="iyy_5" value="${2563.079*unit_factor}" />
-    <xacro:property name="iyy_6" value="${851.576*unit_factor}" />
+    <xacro:property name="iyy_6" value="${226.642*unit_factor}" />
     <xacro:property name="izz_1" value="${11970.081*unit_factor}" />
     <xacro:property name="izz_2" value="${212473.4246*unit_factor}" />
@@ -63,5 +63,5 @@
     <xacro:property name="izz_4" value="${2643.21*unit_factor}" />
     <xacro:property name="izz_5" value="${2643.21*unit_factor}" />
-    <xacro:property name="izz_6" value="${959.69*unit_factor}" />
+    <xacro:property name="izz_6" value="${286.595*unit_factor}" />
 <!--LinkDescription-->
   <link name="${prefix}link_0">
