Commit message: 1.12.2 Update TM5-700 series Xacro, URDF interia parameters.

File: tm_description/urdf/tm5-700-nominal.urdf (robot description, URDF)
Before this commit: robot tm5-700, 9 links, 8 joints
Links:
- link link_2: mass 8.567 -> 8.897
- link link_3: mass 2.273 -> 2.443

File: tm_description/urdf/tm5x-700-nominal.urdf (robot description, URDF)
Before this commit: robot tm5x-700, 9 links, 8 joints
Links:
- link link_2: mass 8.567 -> 8.897
- link link_3: mass 2.273 -> 2.443

File: tm_description/xacro/macro.tm5-700-nominal.urdf.xacro (robot description, xacro)
@@ -40,6 +40,6 @@
     <xacro:property name="mass_0" value="1.000" />
     <xacro:property name="mass_1" value="4.032" />
-    <xacro:property name="mass_2" value="8.567" />
-    <xacro:property name="mass_3" value="2.273" />
+    <xacro:property name="mass_2" value="8.897" />
+    <xacro:property name="mass_3" value="2.443" />
     <xacro:property name="mass_4" value="1.576" />
     <xacro:property name="mass_5" value="1.576" />
@@ -47,18 +47,18 @@
     <xacro:property name="unit_factor" value="0.000001"/>
     <xacro:property name="ixx_1" value="${8800.119*unit_factor}" />
-    <xacro:property name="ixx_2" value="${23552.072*unit_factor}" />
-    <xacro:property name="ixx_3" value="${3380.181*unit_factor}" />
+    <xacro:property name="ixx_2" value="${24459.295*unit_factor}" />
+    <xacro:property name="ixx_3" value="${3632.988*unit_factor}" />
     <xacro:property name="ixx_4" value="${2058.405*unit_factor}" />
     <xacro:property name="ixx_5" value="${2058.405*unit_factor}" />
     <xacro:property name="ixx_6" value="${476.643*unit_factor}" />
     <xacro:property name="iyy_1" value="${11548.982*unit_factor}" />
-    <xacro:property name="iyy_2" value="${198251.97*unit_factor}" />
-    <xacro:property name="iyy_3" value="${33829.144*unit_factor}" />
+    <xacro:property name="iyy_2" value="${205888.616*unit_factor}" />
+    <xacro:property name="iyy_3" value="${36359.26*unit_factor}" />
     <xacro:property name="iyy_4" value="${2563.079*unit_factor}" />
     <xacro:property name="iyy_5" value="${2563.079*unit_factor}" />
     <xacro:property name="iyy_6" value="${851.576*unit_factor}" />
     <xacro:property name="izz_1" value="${11970.081*unit_factor}" />
-    <xacro:property name="izz_2" value="${204592.54*unit_factor}" />
-    <xacro:property name="izz_3" value="${34328.203*unit_factor}" />
+    <xacro:property name="izz_2" value="${212473.4246*unit_factor}" />
+    <xacro:property name="izz_3" value="${36895.644*unit_factor}" />
     <xacro:property name="izz_4" value="${2643.21*unit_factor}" />
     <xacro:property name="izz_5" value="${2643.21*unit_factor}" />

File: tm_description/xacro/macro.tm5x-700-nominal.urdf.xacro (robot description, xacro)
@@ -40,6 +40,6 @@
     <xacro:property name="mass_0" value="1.000" />
     <xacro:property name="mass_1" value="4.032" />
-    <xacro:property name="mass_2" value="8.567" />
-    <xacro:property name="mass_3" value="2.273" />
+    <xacro:property name="mass_2" value="8.897" />
+    <xacro:property name="mass_3" value="2.443" />
     <xacro:property name="mass_4" value="1.576" />
     <xacro:property name="mass_5" value="1.576" />
@@ -47,18 +47,18 @@
     <xacro:property name="unit_factor" value="0.000001"/>
     <xacro:property name="ixx_1" value="${8800.119*unit_factor}" />
-    <xacro:property name="ixx_2" value="${23552.072*unit_factor}" />
-    <xacro:property name="ixx_3" value="${3380.181*unit_factor}" />
+    <xacro:property name="ixx_2" value="${24459.295*unit_factor}" />
+    <xacro:property name="ixx_3" value="${3632.988*unit_factor}" />
     <xacro:property name="ixx_4" value="${2058.405*unit_factor}" />
     <xacro:property name="ixx_5" value="${2058.405*unit_factor}" />
     <xacro:property name="ixx_6" value="${476.643*unit_factor}" />
     <xacro:property name="iyy_1" value="${11548.982*unit_factor}" />
-    <xacro:property name="iyy_2" value="${198251.97*unit_factor}" />
-    <xacro:property name="iyy_3" value="${33829.144*unit_factor}" />
+    <xacro:property name="iyy_2" value="${205888.616*unit_factor}" />
+    <xacro:property name="iyy_3" value="${36359.26*unit_factor}" />
     <xacro:property name="iyy_4" value="${2563.079*unit_factor}" />
     <xacro:property name="iyy_5" value="${2563.079*unit_factor}" />
     <xacro:property name="iyy_6" value="${851.576*unit_factor}" />
     <xacro:property name="izz_1" value="${11970.081*unit_factor}" />
-    <xacro:property name="izz_2" value="${204592.54*unit_factor}" />
-    <xacro:property name="izz_3" value="${34328.203*unit_factor}" />
+    <xacro:property name="izz_2" value="${212473.4246*unit_factor}" />
+    <xacro:property name="izz_3" value="${36895.644*unit_factor}" />
     <xacro:property name="izz_4" value="${2643.21*unit_factor}" />
     <xacro:property name="izz_5" value="${2643.21*unit_factor}" />

Commit message: 1.12.3 Update TM5-900,TM5-700 series Xacro, URDF interia parameters.

File: tm_description/urdf/tm5-700-nominal.urdf (robot description, URDF)
Before this commit: robot tm5-700, 9 links, 8 joints
Links:
- link link_2: mass 8.897 -> 8.567
- link link_3: mass 2.443 -> 2.273

File: tm_description/urdf/tm5-900-nominal.urdf (robot description, URDF)
Before this commit: robot tm5-900, 9 links, 8 joints
Links:
- link link_2: mass 8.567 -> 8.897
- link link_3: mass 2.273 -> 2.443

File: tm_description/urdf/tm5x-700-nominal.urdf (robot description, URDF)
Before this commit: robot tm5x-700, 9 links, 8 joints
Links:
- link link_2: mass 8.897 -> 8.567
- link link_3: mass 2.443 -> 2.273

File: tm_description/urdf/tm5x-900-nominal.urdf (robot description, URDF)
Before this commit: robot tm5x-900, 9 links, 8 joints
Links:
- link link_2: mass 8.567 -> 8.897
- link link_3: mass 2.273 -> 2.443

File: tm_description/xacro/macro.tm5-700-nominal.urdf.xacro (robot description, xacro)
@@ -40,6 +40,6 @@
     <xacro:property name="mass_0" value="1.000" />
     <xacro:property name="mass_1" value="4.032" />
-    <xacro:property name="mass_2" value="8.897" />
-    <xacro:property name="mass_3" value="2.443" />
+    <xacro:property name="mass_2" value="8.567" />
+    <xacro:property name="mass_3" value="2.273" />
     <xacro:property name="mass_4" value="1.576" />
     <xacro:property name="mass_5" value="1.576" />
@@ -47,18 +47,18 @@
     <xacro:property name="unit_factor" value="0.000001"/>
     <xacro:property name="ixx_1" value="${8800.119*unit_factor}" />
-    <xacro:property name="ixx_2" value="${24459.295*unit_factor}" />
-    <xacro:property name="ixx_3" value="${3632.988*unit_factor}" />
+    <xacro:property name="ixx_2" value="${23552.072*unit_factor}" />
+    <xacro:property name="ixx_3" value="${3380.181*unit_factor}" />
     <xacro:property name="ixx_4" value="${2058.405*unit_factor}" />
     <xacro:property name="ixx_5" value="${2058.405*unit_factor}" />
     <xacro:property name="ixx_6" value="${476.643*unit_factor}" />
     <xacro:property name="iyy_1" value="${11548.982*unit_factor}" />
-    <xacro:property name="iyy_2" value="${205888.616*unit_factor}" />
-    <xacro:property name="iyy_3" value="${36359.26*unit_factor}" />
+    <xacro:property name="iyy_2" value="${198251.97*unit_factor}" />
+    <xacro:property name="iyy_3" value="${33829.144*unit_factor}" />
     <xacro:property name="iyy_4" value="${2563.079*unit_factor}" />
     <xacro:property name="iyy_5" value="${2563.079*unit_factor}" />
     <xacro:property name="iyy_6" value="${851.576*unit_factor}" />
     <xacro:property name="izz_1" value="${11970.081*unit_factor}" />
-    <xacro:property name="izz_2" value="${212473.4246*unit_factor}" />
-    <xacro:property name="izz_3" value="${36895.644*unit_factor}" />
+    <xacro:property name="izz_2" value="${204592.54*unit_factor}" />
+    <xacro:property name="izz_3" value="${34328.203*unit_factor}" />
     <xacro:property name="izz_4" value="${2643.21*unit_factor}" />
     <xacro:property name="izz_5" value="${2643.21*unit_factor}" />

File: tm_description/xacro/macro.tm5-900-nominal.urdf.xacro (robot description, xacro)
@@ -40,6 +40,6 @@
     <xacro:property name="mass_0" value="1.000" />
     <xacro:property name="mass_1" value="4.032" />
-    <xacro:property name="mass_2" value="8.567" />
-    <xacro:property name="mass_3" value="2.273" />
+    <xacro:property name="mass_2" value="8.897" />
+    <xacro:property name="mass_3" value="2.443" />
     <xacro:property name="mass_4" value="1.576" />
     <xacro:property name="mass_5" value="1.576" />
@@ -47,18 +47,18 @@
     <xacro:property name="unit_factor" value="0.000001"/>
     <xacro:property name="ixx_1" value="${8800.119*unit_factor}" />
-    <xacro:property name="ixx_2" value="${23552.072*unit_factor}" />
-    <xacro:property name="ixx_3" value="${3380.181*unit_factor}" />
+    <xacro:property name="ixx_2" value="${24459.295*unit_factor}" />
+    <xacro:property name="ixx_3" value="${3632.988*unit_factor}" />
     <xacro:property name="ixx_4" value="${2058.405*unit_factor}" />
     <xacro:property name="ixx_5" value="${2058.405*unit_factor}" />
     <xacro:property name="ixx_6" value="${476.643*unit_factor}" />
     <xacro:property name="iyy_1" value="${11548.982*unit_factor}" />
-    <xacro:property name="iyy_2" value="${198251.97*unit_factor}" />
-    <xacro:property name="iyy_3" value="${33829.144*unit_factor}" />
+    <xacro:property name="iyy_2" value="${205888.616*unit_factor}" />
+    <xacro:property name="iyy_3" value="${36359.26*unit_factor}" />
     <xacro:property name="iyy_4" value="${2563.079*unit_factor}" />
     <xacro:property name="iyy_5" value="${2563.079*unit_factor}" />
     <xacro:property name="iyy_6" value="${851.576*unit_factor}" />
     <xacro:property name="izz_1" value="${11970.081*unit_factor}" />
-    <xacro:property name="izz_2" value="${204592.54*unit_factor}" />
-    <xacro:property name="izz_3" value="${34328.203*unit_factor}" />
+    <xacro:property name="izz_2" value="${212473.4246*unit_factor}" />
+    <xacro:property name="izz_3" value="${36895.644*unit_factor}" />
     <xacro:property name="izz_4" value="${2643.21*unit_factor}" />
     <xacro:property name="izz_5" value="${2643.21*unit_factor}" />

File: tm_description/xacro/macro.tm5x-700-nominal.urdf.xacro (robot description, xacro)
@@ -40,6 +40,6 @@
     <xacro:property name="mass_0" value="1.000" />
     <xacro:property name="mass_1" value="4.032" />
-    <xacro:property name="mass_2" value="8.897" />
-    <xacro:property name="mass_3" value="2.443" />
+    <xacro:property name="mass_2" value="8.567" />
+    <xacro:property name="mass_3" value="2.273" />
     <xacro:property name="mass_4" value="1.576" />
     <xacro:property name="mass_5" value="1.576" />
@@ -47,18 +47,18 @@
     <xacro:property name="unit_factor" value="0.000001"/>
     <xacro:property name="ixx_1" value="${8800.119*unit_factor}" />
-    <xacro:property name="ixx_2" value="${24459.295*unit_factor}" />
-    <xacro:property name="ixx_3" value="${3632.988*unit_factor}" />
+    <xacro:property name="ixx_2" value="${23552.072*unit_factor}" />
+    <xacro:property name="ixx_3" value="${3380.181*unit_factor}" />
     <xacro:property name="ixx_4" value="${2058.405*unit_factor}" />
     <xacro:property name="ixx_5" value="${2058.405*unit_factor}" />
     <xacro:property name="ixx_6" value="${476.643*unit_factor}" />
     <xacro:property name="iyy_1" value="${11548.982*unit_factor}" />
-    <xacro:property name="iyy_2" value="${205888.616*unit_factor}" />
-    <xacro:property name="iyy_3" value="${36359.26*unit_factor}" />
+    <xacro:property name="iyy_2" value="${198251.97*unit_factor}" />
+    <xacro:property name="iyy_3" value="${33829.144*unit_factor}" />
     <xacro:property name="iyy_4" value="${2563.079*unit_factor}" />
     <xacro:property name="iyy_5" value="${2563.079*unit_factor}" />
     <xacro:property name="iyy_6" value="${851.576*unit_factor}" />
     <xacro:property name="izz_1" value="${11970.081*unit_factor}" />
-    <xacro:property name="izz_2" value="${212473.4246*unit_factor}" />
-    <xacro:property name="izz_3" value="${36895.644*unit_factor}" />
+    <xacro:property name="izz_2" value="${204592.54*unit_factor}" />
+    <xacro:property name="izz_3" value="${34328.203*unit_factor}" />
     <xacro:property name="izz_4" value="${2643.21*unit_factor}" />
     <xacro:property name="izz_5" value="${2643.21*unit_factor}" />

File: tm_description/xacro/macro.tm5x-900-nominal.urdf.xacro (robot description, xacro)
@@ -40,6 +40,6 @@
     <xacro:property name="mass_0" value="1.000" />
     <xacro:property name="mass_1" value="4.032" />
-    <xacro:property name="mass_2" value="8.567" />
-    <xacro:property name="mass_3" value="2.273" />
+    <xacro:property name="mass_2" value="8.897" />
+    <xacro:property name="mass_3" value="2.443" />
     <xacro:property name="mass_4" value="1.576" />
     <xacro:property name="mass_5" value="1.576" />
@@ -47,18 +47,18 @@
     <xacro:property name="unit_factor" value="0.000001"/>
     <xacro:property name="ixx_1" value="${8800.119*unit_factor}" />
-    <xacro:property name="ixx_2" value="${23552.072*unit_factor}" />
-    <xacro:property name="ixx_3" value="${3380.181*unit_factor}" />
+    <xacro:property name="ixx_2" value="${24459.295*unit_factor}" />
+    <xacro:property name="ixx_3" value="${3632.988*unit_factor}" />
     <xacro:property name="ixx_4" value="${2058.405*unit_factor}" />
     <xacro:property name="ixx_5" value="${2058.405*unit_factor}" />
     <xacro:property name="ixx_6" value="${476.643*unit_factor}" />
     <xacro:property name="iyy_1" value="${11548.982*unit_factor}" />
-    <xacro:property name="iyy_2" value="${198251.97*unit_factor}" />
-    <xacro:property name="iyy_3" value="${33829.144*unit_factor}" />
+    <xacro:property name="iyy_2" value="${205888.616*unit_factor}" />
+    <xacro:property name="iyy_3" value="${36359.26*unit_factor}" />
     <xacro:property name="iyy_4" value="${2563.079*unit_factor}" />
     <xacro:property name="iyy_5" value="${2563.079*unit_factor}" />
     <xacro:property name="iyy_6" value="${851.576*unit_factor}" />
     <xacro:property name="izz_1" value="${11970.081*unit_factor}" />
-    <xacro:property name="izz_2" value="${204592.54*unit_factor}" />
-    <xacro:property name="izz_3" value="${34328.203*unit_factor}" />
+    <xacro:property name="izz_2" value="${212473.4246*unit_factor}" />
+    <xacro:property name="izz_3" value="${36895.644*unit_factor}" />
     <xacro:property name="izz_4" value="${2643.21*unit_factor}" />
     <xacro:property name="izz_5" value="${2643.21*unit_factor}" />

Commit message: 1.12.5 modify TM5-900,TM5-700 series nominal DH parameters to nominal Xacro, URDF files.

File: tm_description/urdf/tm5-700-nominal.urdf (robot description, URDF)
Before this commit: robot tm5-700, 9 links, 8 joints
Joints:
- joint joint_1: origin xyz=0.000000 0.000000 0.145100 rpy=0.000000 -0.000000 0.000000 -> xyz=0.000000 0.000000 0.145200 rpy=0.000000 -0.000000 0.000000
- joint joint_4: origin xyz=0.311500 0.000000 -0.122200 rpy=0.000000 -0.000000 1.570796 -> xyz=0.311500 0.000000 -0.122300 rpy=0.000000 -0.000000 1.570796
- joint joint_6: origin xyz=0.000000 -0.114400 0.000000 rpy=1.570796 -0.000000 0.000000 -> xyz=0.000000 -0.113150 0.000000 rpy=1.570796 -0.000000 0.000000

File: tm_description/urdf/tm5-900-nominal.urdf (robot description, URDF)
Before this commit: robot tm5-900, 9 links, 8 joints
Joints:
- joint joint_1: origin xyz=0.000000 0.000000 0.145100 rpy=0.000000 -0.000000 0.000000 -> xyz=0.000000 0.000000 0.145200 rpy=0.000000 -0.000000 0.000000
- joint joint_4: origin xyz=0.411500 0.000000 -0.122200 rpy=0.000000 -0.000000 1.570796 -> xyz=0.411500 0.000000 -0.122300 rpy=0.000000 -0.000000 1.570796
- joint joint_6: origin xyz=0.000000 -0.114400 0.000000 rpy=1.570796 -0.000000 0.000000 -> xyz=0.000000 -0.113150 0.000000 rpy=1.570796 -0.000000 0.000000

File: tm_description/urdf/tm5-900.urdf (robot description, URDF)
Before this commit: robot tm5-900, 9 links, 8 joints
Joints:
- joint joint_1: origin xyz=0.000000 0.000000 0.145100 rpy=0.000000 -0.000000 0.000000 -> xyz=0.000000 0.000000 0.145200 rpy=0.000000 -0.000000 0.000000
- joint joint_4: origin xyz=0.411500 0.000000 -0.122200 rpy=0.000000 -0.000000 1.570796 -> xyz=0.411500 0.000000 -0.122300 rpy=0.000000 -0.000000 1.570796
- joint joint_6: origin xyz=0.000000 -0.114400 0.000000 rpy=1.570796 -0.000000 0.000000 -> xyz=0.000000 -0.113150 0.000000 rpy=1.570796 -0.000000 0.000000

File: tm_description/urdf/tm5x-700-nominal.urdf (robot description, URDF)
Before this commit: robot tm5x-700, 9 links, 8 joints
Joints:
- joint joint_1: origin xyz=0.000000 0.000000 0.145100 rpy=0.000000 -0.000000 0.000000 -> xyz=0.000000 0.000000 0.145200 rpy=0.000000 -0.000000 0.000000
- joint joint_4: origin xyz=0.311500 0.000000 -0.122200 rpy=0.000000 -0.000000 1.570796 -> xyz=0.311500 0.000000 -0.122300 rpy=0.000000 -0.000000 1.570796
- joint joint_6: origin xyz=0.000000 -0.114400 0.000000 rpy=1.570796 -0.000000 0.000000 -> xyz=0.000000 -0.113150 0.000000 rpy=1.570796 -0.000000 0.000000

File: tm_description/urdf/tm5x-900-nominal.urdf (robot description, URDF)
Before this commit: robot tm5x-900, 9 links, 8 joints
Joints:
- joint joint_1: origin xyz=0.000000 0.000000 0.145100 rpy=0.000000 -0.000000 0.000000 -> xyz=0.000000 0.000000 0.145200 rpy=0.000000 -0.000000 0.000000
- joint joint_4: origin xyz=0.411500 0.000000 -0.122200 rpy=0.000000 -0.000000 1.570796 -> xyz=0.411500 0.000000 -0.122300 rpy=0.000000 -0.000000 1.570796
- joint joint_6: origin xyz=0.000000 -0.114400 0.000000 rpy=1.570796 -0.000000 0.000000 -> xyz=0.000000 -0.113150 0.000000 rpy=1.570796 -0.000000 0.000000

File: tm_description/xacro/macro.tm5-700-nominal.urdf.xacro (robot description, xacro)
@@ -85,5 +85,5 @@
     <parent link="${prefix}link_0" />
     <child link="${prefix}link_1" />
-    <origin rpy="0.000000 -0.000000 0.000000" xyz="0.000000 0.000000 0.145100" />
+    <origin rpy="0.000000 -0.000000 0.000000" xyz="0.000000 0.000000 0.145200" />
     <axis xyz="0 0 1" />
 <!--limit-->
@@ -175,5 +175,5 @@
     <parent link="${prefix}link_3" />
     <child link="${prefix}link_4" />
-    <origin rpy="0.000000 -0.000000 1.570796" xyz="0.311500 0.000000 -0.122200" />
+    <origin rpy="0.000000 -0.000000 1.570796" xyz="0.311500 0.000000 -0.122300" />
     <axis xyz="0 0 1" />
 <!--limit-->
@@ -235,5 +235,5 @@
     <parent link="${prefix}link_5" />
     <child link="${prefix}link_6" />
-    <origin rpy="1.570796 -0.000000 0.000000" xyz="0.000000 -0.114400 0.000000" />
+    <origin rpy="1.570796 -0.000000 0.000000" xyz="0.000000 -0.113150 0.000000" />
     <axis xyz="0 0 1" />
 <!--limit-->

File: tm_description/xacro/macro.tm5-900-nominal.urdf.xacro (robot description, xacro)
@@ -85,5 +85,5 @@
     <parent link="${prefix}link_0" />
     <child link="${prefix}link_1" />
-    <origin rpy="0.000000 -0.000000 0.000000" xyz="0.000000 0.000000 0.145100" />
+    <origin rpy="0.000000 -0.000000 0.000000" xyz="0.000000 0.000000 0.145200" />
     <axis xyz="0 0 1" />
 <!--limit-->
@@ -175,5 +175,5 @@
     <parent link="${prefix}link_3" />
     <child link="${prefix}link_4" />
-    <origin rpy="0.000000 -0.000000 1.570796" xyz="0.411500 0.000000 -0.122200" />
+    <origin rpy="0.000000 -0.000000 1.570796" xyz="0.411500 0.000000 -0.122300" />
     <axis xyz="0 0 1" />
 <!--limit-->
@@ -235,5 +235,5 @@
     <parent link="${prefix}link_5" />
     <child link="${prefix}link_6" />
-    <origin rpy="1.570796 -0.000000 0.000000" xyz="0.000000 -0.114400 0.000000" />
+    <origin rpy="1.570796 -0.000000 0.000000" xyz="0.000000 -0.113150 0.000000" />
     <axis xyz="0 0 1" />
 <!--limit-->

File: tm_description/xacro/macro.tm5x-700-nominal.urdf.xacro (robot description, xacro)
@@ -85,5 +85,5 @@
     <parent link="${prefix}link_0" />
     <child link="${prefix}link_1" />
-    <origin rpy="0.000000 -0.000000 0.000000" xyz="0.000000 0.000000 0.145100" />
+    <origin rpy="0.000000 -0.000000 0.000000" xyz="0.000000 0.000000 0.145200" />
     <axis xyz="0 0 1" />
 <!--limit-->
@@ -175,5 +175,5 @@
     <parent link="${prefix}link_3" />
     <child link="${prefix}link_4" />
-    <origin rpy="0.000000 -0.000000 1.570796" xyz="0.311500 0.000000 -0.122200" />
+    <origin rpy="0.000000 -0.000000 1.570796" xyz="0.311500 0.000000 -0.122300" />
     <axis xyz="0 0 1" />
 <!--limit-->
@@ -235,5 +235,5 @@
     <parent link="${prefix}link_5" />
     <child link="${prefix}link_6" />
-    <origin rpy="1.570796 -0.000000 0.000000" xyz="0.000000 -0.114400 0.000000" />
+    <origin rpy="1.570796 -0.000000 0.000000" xyz="0.000000 -0.113150 0.000000" />
     <axis xyz="0 0 1" />
 <!--limit-->

File: tm_description/xacro/macro.tm5x-900-nominal.urdf.xacro (robot description, xacro)
@@ -85,5 +85,5 @@
     <parent link="${prefix}link_0" />
     <child link="${prefix}link_1" />
-    <origin rpy="0.000000 -0.000000 0.000000" xyz="0.000000 0.000000 0.145100" />
+    <origin rpy="0.000000 -0.000000 0.000000" xyz="0.000000 0.000000 0.145200" />
     <axis xyz="0 0 1" />
 <!--limit-->
@@ -175,5 +175,5 @@
     <parent link="${prefix}link_3" />
     <child link="${prefix}link_4" />
-    <origin rpy="0.000000 -0.000000 1.570796" xyz="0.411500 0.000000 -0.122200" />
+    <origin rpy="0.000000 -0.000000 1.570796" xyz="0.411500 0.000000 -0.122300" />
     <axis xyz="0 0 1" />
 <!--limit-->
@@ -235,5 +235,5 @@
     <parent link="${prefix}link_5" />
     <child link="${prefix}link_6" />
-    <origin rpy="1.570796 -0.000000 0.000000" xyz="0.000000 -0.114400 0.000000" />
+    <origin rpy="1.570796 -0.000000 0.000000" xyz="0.000000 -0.113150 0.000000" />
     <axis xyz="0 0 1" />
 <!--limit-->
