Commit message: 1.12.15 modify the joint range value of J1,J2,J4,J5,J6 of the eyeless urdf,xacro models and update README.md.

File: tm_description/urdf/tm12x-nominal.urdf (robot description, URDF)
Before this commit: robot tm12x, 9 links, 8 joints
Joints:
- joint joint_1: limit lower=-4.71238898038469 upper=4.71238898038469 effort=353 velocity=2.0943951023931953 -> lower=-6.283185307179586 upper=6.283185307179586 effort=353 velocity=2.0943951023931953
- joint joint_2: limit lower=-3.141592653589793 upper=3.141592653589793 effort=353 velocity=2.0943951023931953 -> lower=-6.283185307179586 upper=6.283185307179586 effort=353 velocity=2.0943951023931953
- joint joint_4: limit lower=-3.141592653589793 upper=3.141592653589793 effort=54 velocity=3.141592653589793 -> lower=-6.283185307179586 upper=6.283185307179586 effort=54 velocity=3.141592653589793
- joint joint_5: limit lower=-3.141592653589793 upper=3.141592653589793 effort=54 velocity=3.141592653589793 -> lower=-6.283185307179586 upper=6.283185307179586 effort=54 velocity=3.141592653589793
- joint joint_6: limit lower=-4.71238898038469 upper=4.71238898038469 effort=54 velocity=3.141592653589793 -> lower=-6.283185307179586 upper=6.283185307179586 effort=54 velocity=3.141592653589793

File: tm_description/urdf/tm14x-nominal.urdf (robot description, URDF)
Before this commit: robot tm14x, 9 links, 8 joints
Joints:
- joint joint_1: limit lower=-4.71238898038469 upper=4.71238898038469 effort=353 velocity=2.0943951023931953 -> lower=-6.283185307179586 upper=6.283185307179586 effort=353 velocity=2.0943951023931953
- joint joint_2: limit lower=-3.141592653589793 upper=3.141592653589793 effort=353 velocity=2.0943951023931953 -> lower=-6.283185307179586 upper=6.283185307179586 effort=353 velocity=2.0943951023931953
- joint joint_4: limit lower=-3.141592653589793 upper=3.141592653589793 effort=54 velocity=2.6179938779914944 -> lower=-6.283185307179586 upper=6.283185307179586 effort=54 velocity=2.6179938779914944
- joint joint_5: limit lower=-3.141592653589793 upper=3.141592653589793 effort=54 velocity=2.6179938779914944 -> lower=-6.283185307179586 upper=6.283185307179586 effort=54 velocity=2.6179938779914944
- joint joint_6: limit lower=-4.71238898038469 upper=4.71238898038469 effort=54 velocity=3.141592653589793 -> lower=-6.283185307179586 upper=6.283185307179586 effort=54 velocity=3.141592653589793

File: tm_description/urdf/tm5x-700-nominal.urdf (robot description, URDF)
Before this commit: robot tm5x-700, 9 links, 8 joints
Joints:
- joint joint_1: limit lower=-4.71238898038469 upper=4.71238898038469 effort=157 velocity=3.141592653589793 -> lower=-6.283185307179586 upper=6.283185307179586 effort=157 velocity=3.141592653589793
- joint joint_2: limit lower=-3.141592653589793 upper=3.141592653589793 effort=157 velocity=3.141592653589793 -> lower=-6.283185307179586 upper=6.283185307179586 effort=157 velocity=3.141592653589793
- joint joint_4: limit lower=-3.141592653589793 upper=3.141592653589793 effort=43 velocity=3.9269908169872414 -> lower=-6.283185307179586 upper=6.283185307179586 effort=43 velocity=3.9269908169872414
- joint joint_5: limit lower=-3.141592653589793 upper=3.141592653589793 effort=43 velocity=3.9269908169872414 -> lower=-6.283185307179586 upper=6.283185307179586 effort=43 velocity=3.9269908169872414
- joint joint_6: limit lower=-4.71238898038469 upper=4.71238898038469 effort=43 velocity=3.9269908169872414 -> lower=-6.283185307179586 upper=6.283185307179586 effort=43 velocity=3.9269908169872414

File: tm_description/urdf/tm5x-900-nominal.urdf (robot description, URDF)
Before this commit: robot tm5x-900, 9 links, 8 joints
Joints:
- joint joint_1: limit lower=-4.71238898038469 upper=4.71238898038469 effort=157 velocity=3.141592653589793 -> lower=-6.283185307179586 upper=6.283185307179586 effort=157 velocity=3.141592653589793
- joint joint_2: limit lower=-3.141592653589793 upper=3.141592653589793 effort=157 velocity=3.141592653589793 -> lower=-6.283185307179586 upper=6.283185307179586 effort=157 velocity=3.141592653589793
- joint joint_4: limit lower=-3.141592653589793 upper=3.141592653589793 effort=43 velocity=3.9269908169872414 -> lower=-6.283185307179586 upper=6.283185307179586 effort=43 velocity=3.9269908169872414
- joint joint_5: limit lower=-3.141592653589793 upper=3.141592653589793 effort=43 velocity=3.9269908169872414 -> lower=-6.283185307179586 upper=6.283185307179586 effort=43 velocity=3.9269908169872414
- joint joint_6: limit lower=-4.71238898038469 upper=4.71238898038469 effort=43 velocity=3.9269908169872414 -> lower=-6.283185307179586 upper=6.283185307179586 effort=43 velocity=3.9269908169872414

File: tm_description/xacro/macro.tm12x-nominal.urdf.xacro (robot description, xacro)
@@ -3,10 +3,10 @@
   <xacro:include filename="$(find tm_description)/xacro/macro.inertial.xacro" />
   <xacro:macro name="tm12x" params="ns prefix color:=none format:=obj
-    joint_1_lower_limit:=${radians(-270)}    joint_1_upper_limit:=${radians(270)}
-    joint_2_lower_limit:=${radians(-180)}    joint_2_upper_limit:=${radians(180)}
+    joint_1_lower_limit:=${radians(-360)}    joint_1_upper_limit:=${radians(360)}
+    joint_2_lower_limit:=${radians(-360)}    joint_2_upper_limit:=${radians(360)}
     joint_3_lower_limit:=${radians(-166)}    joint_3_upper_limit:=${radians(166)}
-    joint_4_lower_limit:=${radians(-180)}    joint_4_upper_limit:=${radians(180)}
-    joint_5_lower_limit:=${radians(-180)}    joint_5_upper_limit:=${radians(180)}
-    joint_6_lower_limit:=${radians(-270)}    joint_6_upper_limit:=${radians(270)}
+    joint_4_lower_limit:=${radians(-360)}    joint_4_upper_limit:=${radians(360)}
+    joint_5_lower_limit:=${radians(-360)}    joint_5_upper_limit:=${radians(360)}
+    joint_6_lower_limit:=${radians(-360)}    joint_6_upper_limit:=${radians(360)}
     joint_1_velocity_limit:=${radians(120)}
     joint_2_velocity_limit:=${radians(120)}

File: tm_description/xacro/macro.tm14x-nominal.urdf.xacro (robot description, xacro)
@@ -3,10 +3,10 @@
   <xacro:include filename="$(find tm_description)/xacro/macro.inertial.xacro" />
   <xacro:macro name="tm14x" params="ns prefix color:=none format:=obj
-    joint_1_lower_limit:=${radians(-270)}    joint_1_upper_limit:=${radians(270)}
-    joint_2_lower_limit:=${radians(-180)}    joint_2_upper_limit:=${radians(180)}
+    joint_1_lower_limit:=${radians(-360)}    joint_1_upper_limit:=${radians(360)}
+    joint_2_lower_limit:=${radians(-360)}    joint_2_upper_limit:=${radians(360)}
     joint_3_lower_limit:=${radians(-163)}    joint_3_upper_limit:=${radians(163)}
-    joint_4_lower_limit:=${radians(-180)}    joint_4_upper_limit:=${radians(180)}
-    joint_5_lower_limit:=${radians(-180)}    joint_5_upper_limit:=${radians(180)}
-    joint_6_lower_limit:=${radians(-270)}    joint_6_upper_limit:=${radians(270)}
+    joint_4_lower_limit:=${radians(-360)}    joint_4_upper_limit:=${radians(360)}
+    joint_5_lower_limit:=${radians(-360)}    joint_5_upper_limit:=${radians(360)}
+    joint_6_lower_limit:=${radians(-360)}    joint_6_upper_limit:=${radians(360)}
     joint_1_velocity_limit:=${radians(120)}
     joint_2_velocity_limit:=${radians(120)}

File: tm_description/xacro/macro.tm5x-700-nominal.urdf.xacro (robot description, xacro)
@@ -3,10 +3,10 @@
   <xacro:include filename="$(find tm_description)/xacro/macro.inertial.xacro" />
   <xacro:macro name="tm5x-700" params="ns prefix color:=none format:=obj
-    joint_1_lower_limit:=${radians(-270)}    joint_1_upper_limit:=${radians(270)}
-    joint_2_lower_limit:=${radians(-180)}    joint_2_upper_limit:=${radians(180)}
+    joint_1_lower_limit:=${radians(-360)}    joint_1_upper_limit:=${radians(360)}
+    joint_2_lower_limit:=${radians(-360)}    joint_2_upper_limit:=${radians(360)}
     joint_3_lower_limit:=${radians(-155)}    joint_3_upper_limit:=${radians(155)}
-    joint_4_lower_limit:=${radians(-180)}    joint_4_upper_limit:=${radians(180)}
-    joint_5_lower_limit:=${radians(-180)}    joint_5_upper_limit:=${radians(180)}
-    joint_6_lower_limit:=${radians(-270)}    joint_6_upper_limit:=${radians(270)}
+    joint_4_lower_limit:=${radians(-360)}    joint_4_upper_limit:=${radians(360)}
+    joint_5_lower_limit:=${radians(-360)}    joint_5_upper_limit:=${radians(360)}
+    joint_6_lower_limit:=${radians(-360)}    joint_6_upper_limit:=${radians(360)}
     joint_1_velocity_limit:=${radians(180)}
     joint_2_velocity_limit:=${radians(180)}

File: tm_description/xacro/macro.tm5x-900-nominal.urdf.xacro (robot description, xacro)
@@ -3,10 +3,10 @@
   <xacro:include filename="$(find tm_description)/xacro/macro.inertial.xacro" />
   <xacro:macro name="tm5x-900" params="ns prefix color:=none format:=obj
-    joint_1_lower_limit:=${radians(-270)}    joint_1_upper_limit:=${radians(270)}
-    joint_2_lower_limit:=${radians(-180)}    joint_2_upper_limit:=${radians(180)}
+    joint_1_lower_limit:=${radians(-360)}    joint_1_upper_limit:=${radians(360)}
+    joint_2_lower_limit:=${radians(-360)}    joint_2_upper_limit:=${radians(360)}
     joint_3_lower_limit:=${radians(-155)}    joint_3_upper_limit:=${radians(155)}
-    joint_4_lower_limit:=${radians(-180)}    joint_4_upper_limit:=${radians(180)}
-    joint_5_lower_limit:=${radians(-180)}    joint_5_upper_limit:=${radians(180)}
-    joint_6_lower_limit:=${radians(-270)}    joint_6_upper_limit:=${radians(270)}
+    joint_4_lower_limit:=${radians(-360)}    joint_4_upper_limit:=${radians(360)}
+    joint_5_lower_limit:=${radians(-360)}    joint_5_upper_limit:=${radians(360)}
+    joint_6_lower_limit:=${radians(-360)}    joint_6_upper_limit:=${radians(360)}
     joint_1_velocity_limit:=${radians(180)}
     joint_2_velocity_limit:=${radians(180)}

Commit message: 1.0.0 Initial version of TM Humble ROS2 application.

File: tm_description/urdf/tm12x-nominal.urdf (robot description, URDF)
Before this commit: robot tm12x, 9 links, 8 joints
Joints:
- joint joint_1: limit lower=-6.283185307179586 upper=6.283185307179586 effort=353 velocity=2.0943951023931953 -> lower=-4.71238898038469 upper=4.71238898038469 effort=353 velocity=2.0943951023931953
- joint joint_2: limit lower=-6.283185307179586 upper=6.283185307179586 effort=353 velocity=2.0943951023931953 -> lower=-3.141592653589793 upper=3.141592653589793 effort=353 velocity=2.0943951023931953
- joint joint_4: limit lower=-6.283185307179586 upper=6.283185307179586 effort=54 velocity=3.141592653589793 -> lower=-3.141592653589793 upper=3.141592653589793 effort=54 velocity=3.141592653589793
- joint joint_5: limit lower=-6.283185307179586 upper=6.283185307179586 effort=54 velocity=3.141592653589793 -> lower=-3.141592653589793 upper=3.141592653589793 effort=54 velocity=3.141592653589793
- joint joint_6: limit lower=-6.283185307179586 upper=6.283185307179586 effort=54 velocity=3.141592653589793 -> lower=-4.71238898038469 upper=4.71238898038469 effort=54 velocity=3.141592653589793

File: tm_description/urdf/tm14x-nominal.urdf (robot description, URDF)
Before this commit: robot tm14x, 9 links, 8 joints
Joints:
- joint joint_1: limit lower=-6.283185307179586 upper=6.283185307179586 effort=353 velocity=2.0943951023931953 -> lower=-4.71238898038469 upper=4.71238898038469 effort=353 velocity=2.0943951023931953
- joint joint_2: limit lower=-6.283185307179586 upper=6.283185307179586 effort=353 velocity=2.0943951023931953 -> lower=-3.141592653589793 upper=3.141592653589793 effort=353 velocity=2.0943951023931953
- joint joint_4: limit lower=-6.283185307179586 upper=6.283185307179586 effort=54 velocity=2.6179938779914944 -> lower=-3.141592653589793 upper=3.141592653589793 effort=54 velocity=2.6179938779914944
- joint joint_5: limit lower=-6.283185307179586 upper=6.283185307179586 effort=54 velocity=2.6179938779914944 -> lower=-3.141592653589793 upper=3.141592653589793 effort=54 velocity=2.6179938779914944
- joint joint_6: limit lower=-6.283185307179586 upper=6.283185307179586 effort=54 velocity=3.141592653589793 -> lower=-4.71238898038469 upper=4.71238898038469 effort=54 velocity=3.141592653589793

File: tm_description/urdf/tm5x-700-nominal.urdf (robot description, URDF)
Before this commit: robot tm5x-700, 9 links, 8 joints
Joints:
- joint joint_1: limit lower=-6.283185307179586 upper=6.283185307179586 effort=157 velocity=3.141592653589793 -> lower=-4.71238898038469 upper=4.71238898038469 effort=157 velocity=3.141592653589793
- joint joint_2: limit lower=-6.283185307179586 upper=6.283185307179586 effort=157 velocity=3.141592653589793 -> lower=-3.141592653589793 upper=3.141592653589793 effort=157 velocity=3.141592653589793
- joint joint_4: limit lower=-6.283185307179586 upper=6.283185307179586 effort=43 velocity=3.9269908169872414 -> lower=-3.141592653589793 upper=3.141592653589793 effort=43 velocity=3.9269908169872414
- joint joint_5: limit lower=-6.283185307179586 upper=6.283185307179586 effort=43 velocity=3.9269908169872414 -> lower=-3.141592653589793 upper=3.141592653589793 effort=43 velocity=3.9269908169872414
- joint joint_6: limit lower=-6.283185307179586 upper=6.283185307179586 effort=43 velocity=3.9269908169872414 -> lower=-4.71238898038469 upper=4.71238898038469 effort=43 velocity=3.9269908169872414

File: tm_description/urdf/tm5x-900-nominal.urdf (robot description, URDF)
Before this commit: robot tm5x-900, 9 links, 8 joints
Joints:
- joint joint_1: limit lower=-6.283185307179586 upper=6.283185307179586 effort=157 velocity=3.141592653589793 -> lower=-4.71238898038469 upper=4.71238898038469 effort=157 velocity=3.141592653589793
- joint joint_2: limit lower=-6.283185307179586 upper=6.283185307179586 effort=157 velocity=3.141592653589793 -> lower=-3.141592653589793 upper=3.141592653589793 effort=157 velocity=3.141592653589793
- joint joint_4: limit lower=-6.283185307179586 upper=6.283185307179586 effort=43 velocity=3.9269908169872414 -> lower=-3.141592653589793 upper=3.141592653589793 effort=43 velocity=3.9269908169872414
- joint joint_5: limit lower=-6.283185307179586 upper=6.283185307179586 effort=43 velocity=3.9269908169872414 -> lower=-3.141592653589793 upper=3.141592653589793 effort=43 velocity=3.9269908169872414
- joint joint_6: limit lower=-6.283185307179586 upper=6.283185307179586 effort=43 velocity=3.9269908169872414 -> lower=-4.71238898038469 upper=4.71238898038469 effort=43 velocity=3.9269908169872414

File: tm_description/xacro/macro.tm12x-nominal.urdf.xacro (robot description, xacro)
@@ -3,10 +3,10 @@
   <xacro:include filename="$(find tm_description)/xacro/macro.inertial.xacro" />
   <xacro:macro name="tm12x" params="ns prefix color:=none format:=obj
-    joint_1_lower_limit:=${radians(-360)}    joint_1_upper_limit:=${radians(360)}
-    joint_2_lower_limit:=${radians(-360)}    joint_2_upper_limit:=${radians(360)}
+    joint_1_lower_limit:=${radians(-270)}    joint_1_upper_limit:=${radians(270)}
+    joint_2_lower_limit:=${radians(-180)}    joint_2_upper_limit:=${radians(180)}
     joint_3_lower_limit:=${radians(-166)}    joint_3_upper_limit:=${radians(166)}
-    joint_4_lower_limit:=${radians(-360)}    joint_4_upper_limit:=${radians(360)}
-    joint_5_lower_limit:=${radians(-360)}    joint_5_upper_limit:=${radians(360)}
-    joint_6_lower_limit:=${radians(-360)}    joint_6_upper_limit:=${radians(360)}
+    joint_4_lower_limit:=${radians(-180)}    joint_4_upper_limit:=${radians(180)}
+    joint_5_lower_limit:=${radians(-180)}    joint_5_upper_limit:=${radians(180)}
+    joint_6_lower_limit:=${radians(-270)}    joint_6_upper_limit:=${radians(270)}
     joint_1_velocity_limit:=${radians(120)}
     joint_2_velocity_limit:=${radians(120)}

File: tm_description/xacro/macro.tm14x-nominal.urdf.xacro (robot description, xacro)
@@ -3,10 +3,10 @@
   <xacro:include filename="$(find tm_description)/xacro/macro.inertial.xacro" />
   <xacro:macro name="tm14x" params="ns prefix color:=none format:=obj
-    joint_1_lower_limit:=${radians(-360)}    joint_1_upper_limit:=${radians(360)}
-    joint_2_lower_limit:=${radians(-360)}    joint_2_upper_limit:=${radians(360)}
+    joint_1_lower_limit:=${radians(-270)}    joint_1_upper_limit:=${radians(270)}
+    joint_2_lower_limit:=${radians(-180)}    joint_2_upper_limit:=${radians(180)}
     joint_3_lower_limit:=${radians(-163)}    joint_3_upper_limit:=${radians(163)}
-    joint_4_lower_limit:=${radians(-360)}    joint_4_upper_limit:=${radians(360)}
-    joint_5_lower_limit:=${radians(-360)}    joint_5_upper_limit:=${radians(360)}
-    joint_6_lower_limit:=${radians(-360)}    joint_6_upper_limit:=${radians(360)}
+    joint_4_lower_limit:=${radians(-180)}    joint_4_upper_limit:=${radians(180)}
+    joint_5_lower_limit:=${radians(-180)}    joint_5_upper_limit:=${radians(180)}
+    joint_6_lower_limit:=${radians(-270)}    joint_6_upper_limit:=${radians(270)}
     joint_1_velocity_limit:=${radians(120)}
     joint_2_velocity_limit:=${radians(120)}

File: tm_description/xacro/macro.tm5x-700-nominal.urdf.xacro (robot description, xacro)
@@ -3,10 +3,10 @@
   <xacro:include filename="$(find tm_description)/xacro/macro.inertial.xacro" />
   <xacro:macro name="tm5x-700" params="ns prefix color:=none format:=obj
-    joint_1_lower_limit:=${radians(-360)}    joint_1_upper_limit:=${radians(360)}
-    joint_2_lower_limit:=${radians(-360)}    joint_2_upper_limit:=${radians(360)}
+    joint_1_lower_limit:=${radians(-270)}    joint_1_upper_limit:=${radians(270)}
+    joint_2_lower_limit:=${radians(-180)}    joint_2_upper_limit:=${radians(180)}
     joint_3_lower_limit:=${radians(-155)}    joint_3_upper_limit:=${radians(155)}
-    joint_4_lower_limit:=${radians(-360)}    joint_4_upper_limit:=${radians(360)}
-    joint_5_lower_limit:=${radians(-360)}    joint_5_upper_limit:=${radians(360)}
-    joint_6_lower_limit:=${radians(-360)}    joint_6_upper_limit:=${radians(360)}
+    joint_4_lower_limit:=${radians(-180)}    joint_4_upper_limit:=${radians(180)}
+    joint_5_lower_limit:=${radians(-180)}    joint_5_upper_limit:=${radians(180)}
+    joint_6_lower_limit:=${radians(-270)}    joint_6_upper_limit:=${radians(270)}
     joint_1_velocity_limit:=${radians(180)}
     joint_2_velocity_limit:=${radians(180)}

File: tm_description/xacro/macro.tm5x-900-nominal.urdf.xacro (robot description, xacro)
@@ -3,10 +3,10 @@
   <xacro:include filename="$(find tm_description)/xacro/macro.inertial.xacro" />
   <xacro:macro name="tm5x-900" params="ns prefix color:=none format:=obj
-    joint_1_lower_limit:=${radians(-360)}    joint_1_upper_limit:=${radians(360)}
-    joint_2_lower_limit:=${radians(-360)}    joint_2_upper_limit:=${radians(360)}
+    joint_1_lower_limit:=${radians(-270)}    joint_1_upper_limit:=${radians(270)}
+    joint_2_lower_limit:=${radians(-180)}    joint_2_upper_limit:=${radians(180)}
     joint_3_lower_limit:=${radians(-155)}    joint_3_upper_limit:=${radians(155)}
-    joint_4_lower_limit:=${radians(-360)}    joint_4_upper_limit:=${radians(360)}
-    joint_5_lower_limit:=${radians(-360)}    joint_5_upper_limit:=${radians(360)}
-    joint_6_lower_limit:=${radians(-360)}    joint_6_upper_limit:=${radians(360)}
+    joint_4_lower_limit:=${radians(-180)}    joint_4_upper_limit:=${radians(180)}
+    joint_5_lower_limit:=${radians(-180)}    joint_5_upper_limit:=${radians(180)}
+    joint_6_lower_limit:=${radians(-270)}    joint_6_upper_limit:=${radians(270)}
     joint_1_velocity_limit:=${radians(180)}
     joint_2_velocity_limit:=${radians(180)}
