Commit message: 1.12.1 Add TM other series Xacro, URDF robort models and related moveit demo launch files.

File: tm_description/xacro/macro.materials.xacro (robot description, xacro)
@@ -2,4 +2,7 @@
 <robot xmlns:xacro="http://www.ros.org/wiki/xacro">
 	<xacro:macro name="tmr_materials">
+		<material name="none">
+			<color rgba="0.0 0.0 0.0 1.0" />
+		</material>
 		<material name="lightgrey">
 			<color rgba="0.5 0.5 0.5 1.0" />
